Commit message: virtual end effector

File: franka_description/robots/common/franka_robot.xacro (robot description, xacro)
@@ -14,4 +14,10 @@
     <xacro:include filename="$(find franka_description)/robots/common/franka_arm.xacro" />
     <xacro:franka_arm arm_id="${arm_id}" safety_distance="0.03" gazebo="$(arg gazebo)" joint_limits="${joint_limits}"/>
+    <link name="${arm_id}_virtual_EE_link" />
+    <joint name="${arm_id}_virtual_EE_joint" type="fixed">
+      <origin xyz="0 0 0.048" rpy="0 0 0" />
+      <parent link="$(arg arm_id)_link8" />
+      <child link="${arm_id}_virtual_EE_link" />
+    </joint>
     <xacro:if value="$(arg hand)">
       <xacro:include filename="$(find franka_description)/robots/common/franka_hand.xacro"/>

Commit message: Add virtual EE Z offset as launch parameter

File: franka_description/robots/common/franka_robot.xacro (robot description, xacro)
@@ -16,5 +16,5 @@
     <link name="${arm_id}_virtual_EE_link" />
     <joint name="${arm_id}_virtual_EE_joint" type="fixed">
-      <origin xyz="0 0 0.048" rpy="0 0 0" />
+      <origin xyz="0 0 $(arg base_offset_z)" rpy="0 0 0" />
       <parent link="$(arg arm_id)_link8" />
       <child link="${arm_id}_virtual_EE_link" />
